Commit message: change wheel color

File: pathfinder/description/robot_core.xacro (robot description, xacro)
@@ -54,5 +54,5 @@
                 <cylinder radius="0.05" length="0.04"/>
             </geometry>
-            <material name="black"/>
+            <material name="grey"/>
         </visual>
         <collision>
@@ -66,5 +66,5 @@
     </link>
     <gazebo reference="left_wheel">
-        <material>Gazebo/Black</material>
+        <material>Gazebo/Grey</material>
     </gazebo>
     <!-- RIGHT WHEEL LINK -->
